File: pcb/MontesDeOca_DCI_CEIoT_Final.kicad_pcb (KiCad board)
At the start: 2 copper layers, 45 parts, among them J1 USB CON8, J2 Conn_01x20_MountingPin, J3 Conn_01x20_MountingPin, Q1 S8050(NPN), Q2 S8050(NPN), SW1 SW_MEC_5G, SW2 SW_MEC_5G, U1 AMS1117, U2 CP2102N, U3 ESP32_SIP

Commit message: Actualizacion segun correcciones ralizadas
Se avanzo adicionalmente en el posicionamiento de los componentes, el ruteo y el modelo 3D
Parts:
- C1, C2: footprint Capacitor_SMD:C_0603_1608Metric -> Capacitor_SMD:C_0805_2012Metric
- C10, C3, C4, C5, C6, C7, C8, C9, L1: footprint Capacitor_SMD:C_0402_1005Metric -> Capacitor_SMD:C_0805_2012Metric
- D1: footprint LED_SMD:LED_0603_1608Metric -> LED_SMD:LED_0805_2012Metric
- R1, R10, R11, R12, R13, R14, R15, R16, R17, R18, R2, R3, R4, R5, R6, R7, R8, R9: footprint Resistor_SMD:R_0402_1005Metric -> Resistor_SMD:R_0805_2012Metric
- moved ANT1 67.9 mm to (58.0, 78.0), turned to 90 degrees
- moved U1 61.9 mm to (90.0, 68.5), turned to 180 degrees
- moved C1 58.9 mm to (90.5, 57.5), turned to 180 degrees
- moved D1 58.1 mm to (88.1, 62.5)
- moved L1 57.6 mm to (70.5, 85.0), turned to 90 degrees
- moved C8 57.4 mm to (68.0, 72.0), turned to 270 degrees
- moved R14 54.1 mm to (82.4, 68.0)
- moved C4 51.4 mm to (79.5, 85.0), turned to 270 degrees
- moved C7 48.9 mm to (76.5, 85.0), turned to 270 degrees
- moved C5 48.8 mm to (73.5, 85.0), turned to 90 degrees
- moved J2 48.6 mm to (64.5, 53.0), turned to 90 degrees
- moved R15 47.0 mm to (82.5, 85.1), turned to 270 degrees
- moved C2 44.0 mm to (84.0, 57.5)
- moved R1 40.9 mm to (92.1, 62.5)
- moved Q1 40.1 mm to (104.5, 66.0), turned to 90 degrees
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Connections:
- net CTS renamed Net-(R7-Pad2)
- net RXD renamed Net-(R4-Pad2)
- net TXD renamed Net-(R5-Pad2)
- Q2 pad 2: IO0 -> Net-(Q2-Pad2)
- R17 pad 1: IO0 -> Net-(Q2-Pad2)
Routing:
- net +5V: track 0.00 -> 192.6 mm, vias 0 -> 3
- net GND: track 0.00 -> 55.7 mm, vias 0 -> 15
- net +3.3VDAC: track 0.00 -> 35.7 mm, vias 0 -> 2
- net USB_DN: track 0.00 -> 29.0 mm, vias 0 -> 2
- net USB_DP: track 0.00 -> 26.9 mm, vias 0 -> 2
- net Net-(C9-Pad1): track 0.00 -> 26.0 mm
- net Net-(D3-Pad1): track 0.00 -> 23.6 mm
- net Net-(D2-Pad1): track 0.00 -> 19.9 mm
- net Net-(D4-Pad1): track 0.00 -> 18.3 mm
- net Net-(C10-Pad1): track 0.00 -> 14.6 mm
- net EN: track 0.00 -> 12.1 mm
- net Net-(Q2-Pad2): track 0.00 -> 11.8 mm, vias 0 -> 1
- net Net-(Q2-Pad1): track 0.00 -> 9.11 mm
- net Net-(Q1-Pad1): track 0.00 -> 4.94 mm
- net RTS: track 0.00 -> 4.88 mm
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- added copper zone on B.Cu, net GND
Other:
- board outline added: 116 x 61 mm
- copper layers 2 -> 4
- net class Default: clearance 0.2 -> 0.8; trace_width 0.25 -> 0.8; via_dia 0.8 -> 1.6; via_drill 0.4 -> 0.8
- net class Small added: clearance 0.15, trace_width 0.2, via_dia 1, via_drill 0.6
- rule trace_clearance: 0.2 -> 0.8
- board text added: "INDUSTRIA ARGENTINA @2021 DCI | FIUBA"
- board text added: "Replica ESP32-Pico-Tag by Federico Montes de Oca"

Commit message: Actualizacion
Parts:
- added FID1: Fiducial, Fiducial:Fiducial_0.5mm_Mask1.5mm, F.Cu at (57.5, 96.5)
- added FID2: Fiducial, Fiducial:Fiducial_0.5mm_Mask1.5mm, F.Cu at (57.5, 93.4)
- added FID3: Fiducial, Fiducial:Fiducial_0.5mm_Mask1.5mm, F.Cu at (57.5, 90.4)
