File: pcb/MontesDeOca_DCI_CEIoT_Final.sch (KiCad schematic (older format))
At the start: 45 parts, among them J1 USB CON8, J2 Conn_01x20_MountingPin, J3 Conn_01x20_MountingPin, Q1 S8050(NPN), Q2 S8050(NPN), SW1 SW_MEC_5G, SW2 SW_MEC_5G, U1 AMS1117, U2 CP2102N, U3 ESP32_SIP

Commit message: Actualizacion segun correcciones ralizadas
Se avanzo adicionalmente en el posicionamiento de los componentes, el ruteo y el modelo 3D
Parts:
- C1, C2: footprint Capacitor_SMD:C_0603_1608Metric -> Capacitor_SMD:C_0805_2012Metric
- C10, C3, C4, C5, C6, C7, C8, C9: footprint Capacitor_SMD:C_0402_1005Metric -> Capacitor_SMD:C_0805_2012Metric
- D1: footprint LED_SMD:LED_0603_1608Metric -> LED_SMD:LED_0805_2012Metric
- J1: Catalog (none) -> DigiKey 670-2675-2-ND; Manufacturer Part # (none) -> DX4R005JJ2R1800
- L1: footprint Capacitor_SMD:C_0402_1005Metric -> Capacitor_SMD:C_0805_2012Metric; Catalog (none) -> DigiKey 732-7772-2-ND; Man Model # (none) -> 885012006030; Manufacturer (none) -> Wurth Elektronik
- Q1, Q2: Catalog (none) -> www.Win-Source.Net Catalog#: 1102202-MMSS8050-H-TP
- R1, R10, R11, R12, R13, R14, R15, R16, R17, R18, R2, R3, R4, R5, R6, R7, R8, R9: footprint Resistor_SMD:R_0402_1005Metric -> Resistor_SMD:R_0805_2012Metric
- U1: Catalog (none) -> www. Win-Source.Net catalog #: 094958-AMS1117-3.3
- U2: Catalog (none) -> www.Win-Source.Net Catalog#: 758381-CP2102N-A01-GQFN28
Connections:
- net IO0: no longer Q2.2 (C), R17.1
- net CTS: no longer names the net of R7.2, U2.23 (CTS)
- net RXD: no longer names the net of R4.2, U2.25 (RXD)
- net TXD: no longer names the net of R5.2, U2.26 (TXD)
- new net: Q2.2 (C), R17.1
Other:
- moved on the sheet: R17, R18, R4, R5, R6, R7

Commit message: Actualizacion
Parts:
- added FID1, FID2, FID3: Fiducial, Fiducial:Fiducial_0.5mm_Mask1.5mm, symbol Mechanical:Fiducial
Changed lines of the file:
@@
 Wire Wire Line
 	4800 2300 5450 2300
+$Comp
+L Mechanical:Fiducial FID1
+U 1 1 6141280C
+P 5500 7300
+F 0 "FID1" H 5585 7346 50  0000 L CNN
+F 1 "Fiducial" H 5585 7255 50  0000 L CNN
+F 2 "Fiducial:Fiducial_0.5mm_Mask1.5mm" H 5500 7300 50  0001 C CNN
+F 3 "~" H 5500 7300 50  0001 C CNN
+	1    5500 7300
+	1    0    0    -1
+$EndComp
+$Comp
+L Mechanical:Fiducial FID3
+U 1 1 61412DEC
+P 6050 7300
+F 0 "FID3" H 6135 7346 50  0000 L CNN
+F 1 "Fiducial" H 6135 7255 50  0000 L CNN
+F 2 "Fiducial:Fiducial_0.5mm_Mask1.5mm" H 6050 7300 50  0001 C CNN
+F 3 "~" H 6050 7300 50  0001 C CNN
+	1    6050 7300
+	1    0    0    -1
+$EndComp
+$Comp
+L Mechanical:Fiducial FID2
+U 1 1 61413188
+P 5800 7550
+F 0 "FID2" H 5885 7596 50  0000 L CNN
+F 1 "Fiducial" H 5885 7505 50  0000 L CNN
+F 2 "Fiducial:Fiducial_0.5mm_Mask1.5mm" H 5800 7550 50  0001 C CNN
+F 3 "~" H 5800 7550 50  0001 C CNN
+	1    5800 7550
+	1    0    0    -1
+$EndComp
 $EndSCHEMATC
